File: nano.kicad_pcb (KiCad board)
At the start: 2 copper layers, 183.7 x 126.7 mm, 18 parts

Commit message: Final
Parts:
- added D3: 1N4148WT, Diode_SMD:D_SOD-523, B.Cu at (75.5, 96.5)
- added M1: Motor_DC, Motors:Vybronics_VZ30C1T8219732L, F.Cu at (85.6, 110.2)
- added Q1: BP103, Package_TO_SOT_THT:TO-18-3_Lens, B.Cu at (81.3, 73.7)
- added Q2: NPN, Package_TO_SOT_THT:TO-92L_HandSolder, B.Cu at (109.2, 81.3)
- added Q3: NPN, Package_TO_SOT_THT:TO-92L_HandSolder, F.Cu at (106.7, 101.6)
- added R3: R_Photo, OptoDevice:R_LDR_5.1x4.3mm_P3.4mm_Vertical, F.Cu at (57.6, 167.6)
- added SW1: SW_Push, Button_Switch_THT:SW_PUSH_6mm, F.Cu at (81.9, 92.9)
- D1: value LED -> 1N4148WT; footprint LED_THT:LED_D5.0mm -> Diode_SMD:D_SOD-523; moved to B.Cu
- R1, R2: moved to B.Cu
- moved D2 89.4 mm to (124.5, 137.2), turned to 0 degrees
- moved R1 68.8 mm to (106.7, 170.2), turned to 0 degrees
- moved D1 23.8 mm to (136.5, 91.4)
- moved R2 13.0 mm to (71.1, 109.2), turned to 90 degrees
- turned BT1 to 180 degrees
Connections:
- D1 pad 2: Net-(BT1-+) -> Net-(D1-A)
- D2 pad 2: Net-(BT1-+) -> Net-(D2-A)
- R1 pad 1: Net-(D1-K) -> Net-(BT1-+)
- R1 pad 2: Net-(BT1--) -> Net-(D2-A)
- R2 pad 1: Net-(D2-K) -> Net-(BT1-+)
- R2 pad 2: Net-(BT1--) -> Net-(D3-A)
Routing:
- net Net-(Q1-E): track 0.00 -> 115.6 mm
- net Net-(D1-K): track 21.3 -> 101.5 mm
- net Net-(D3-A): track 0.00 -> 64.3 mm
- net Net-(D2-K): track 29.8 -> 79.5 mm
- net Net-(BT1--): track 122.6 -> 78.6 mm
- net Net-(Q3-E): track 0.00 -> 38.7 mm
- net Net-(D2-A): track 0.00 -> 38.3 mm
- net Net-(D1-A): track 0.00 -> 29.7 mm
- net Net-(Q1-B): track 0.00 -> 28.6 mm
- net Net-(BT1-+): track 156.6 -> 172.6 mm

Commit message: the last
Parts:
- removed the G*** at (86.4, 162.6) (x2)
- removed the G*** at (91.4, 91.4)
- removed the G*** at (132.1, 147.3)
- removed the G*** at (66.0, 162.6) (x2)
- removed the G*** at (127.0, 111.8)
- removed the G*** at (102.7, 84.5)
- removed the G*** at (86.4, 127.0)
- removed the G*** at (127.0, 162.6)
- removed the G*** at (127.4, 76.2)
- removed the G*** at (127.0, 101.6)
- removed Q1: BP103, Package_TO_SOT_THT:TO-18-3_Lens
- removed `: LOGO, LOGO
- added G***: LOGO, LOGO, F.Cu at (96.5, 132.1)
- added G***: LOGO, LOGO, B.Cu at (96.5, 132.1)
- added Q4: BP103, Package_TO_SOT_THT:TO-18-3_Lens, F.Cu at (90.2, 146.1)
- BT1, R1, R2: moved to F.Cu
- Q3, R3, SW1: moved to B.Cu
- moved D3 71.8 mm to (137.9, 132.1)
- moved SW1 67.6 mm to (126.4, 143.7)
- moved R1 66.2 mm to (111.8, 104.1), turned to -90 degrees
- moved M1 61.8 mm to (146.5, 120.4)
- moved D1 59.5 mm to (116.1, 147.3)
- moved R2 56.1 mm to (127.0, 104.1), turned to -90 degrees
- moved Q2 55.9 mm to (111.8, 137.2)
- moved R3 49.1 mm to (91.4, 132.1), turned to -90 degrees
- moved Q3 27.0 mm to (124.5, 121.9), turned to 180 degrees
- moved BT1 25.9 mm to (91.4, 116.8), turned to 90 degrees
- moved D2 18.0 mm to (111.8, 124.5), turned to 90 degrees
Routing:
- net Net-(Q4-E): track 115.6 -> 15.9 mm
- net Net-(BT1-+): track 172.6 -> 102.8 mm
- net Net-(D2-K): track 79.5 -> 30.4 mm
- net Net-(D3-A): track 64.3 -> 27.1 mm
- net Net-(BT1--): track 78.6 -> 49.9 mm
- net Net-(D2-A): track 38.3 -> 10.2 mm
- net Net-(D1-A): track 29.7 -> 9.14 mm
- net Net-(Q3-E): track 38.7 -> 21.7 mm
- net Net-(D1-K): track 101.5 -> 114.0 mm
- net Net-(Q2-B): track 28.6 -> 25.7 mm
Other:
- board size 183.7 x 126.7 mm -> 144.1 x 78.6 mm
