File: nano.kicad_sch (KiCad schematic)
At the start: 5 parts

Commit message: Final
Parts:
- removed D1: LED, LED_THT:LED_D5.0mm, symbol Device:LED
- added D1, D3: 1N4148WT, Diode_SMD:D_SOD-523, symbol Diode:1N4148WT
- added M1: Motor_DC, Motors:Vybronics_VZ30C1T8219732L, symbol Motor:Motor_DC
- added Q1: BP103, Package_TO_SOT_THT:TO-18-3_Lens, symbol Sensor_Optical:BP103
- added Q2, Q3: NPN, Package_TO_SOT_THT:TO-92L_HandSolder, symbol Simulation_SPICE:NPN
- added R3: R_Photo, OptoDevice:R_LDR_5.1x4.3mm_P3.4mm_Vertical, symbol Device:R_Photo
- added SW1: SW_Push, Button_Switch_THT:SW_PUSH_6mm, symbol Switch:SW_Push
Connections:
- net at BT1.1 (+): now also R1.1, R2.1, M1.1 (+); no longer D2.2 (A)
- net at D2.1 (K): now also Q2.1 (C), Q3.2 (B); no longer R2.1
- new net: BT1.2 (-), R3.1
- new net: Q1.1 (E), R3.2
- new net: Q1.2 (B), Q2.2 (B)
- new net: D1.1 (K), D3.1 (K), M1.2 (-), Q1.3 (C), SW1.1
- new net: D3.2 (A), Q3.1 (C), R2.2
- new net: Q3.3 (E), SW1.2
- new net: D2.2 (A), R1.2
- new net: D1.2 (A), Q2.3 (E)
Other:
- moved on the sheet: BT1, D2, R1, R2

Commit message: the last
Parts:
- removed Q1: BP103, Package_TO_SOT_THT:TO-18-3_Lens, symbol Sensor_Optical:BP103
- added Q4: BP103, Package_TO_SOT_THT:TO-18-3_Lens, symbol Sensor_Optical:BP103
Connections:
- net at R3.2: now also Q4.1 (E)
- net at Q2.2 (B): now also Q4.2 (B)
- net at D1.1 (K), D3.1 (K), M1.2 (-)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: now also Q4.3 (C)
Other:
- moved on the sheet: R3
Changed lines of the file:
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@@
-	)
-	(junction
-		(at 121.92 111.76)
-		(diameter 0)
-		(color 0 0 0 0)
 	)
 	(junction
@@
 	(wire
 		(pts
-			(xy 121.92 101.6) (xy 121.92 104.14)
+			(xy 121.92 101.6) (xy 121.92 102.87)
 		)
 		(stroke
@@
 	(wire
 		(pts
-			(xy 129.54 119.38) (xy 129.54 116.84)
+			(xy 129.54 119.38) (xy 129.54 118.11)
 		)
 		(stroke
@@
 	(wire
 		(pts
-			(xy 128.27 119.38) (xy 129.54 119.38)
+			(xy 129.54 119.38) (xy 128.27 119.38)
+		)
+		(stroke
+			(width 0)
+			(type default)
+		)
+	)
+	(wire
+		(pts
+			(xy 121.92 110.49) (xy 121.92 113.03)
 		)
 		(stroke
@@
 	(wire
 		(pts
-			(xy 121.92 121.92) (xy 121.92 135.89)
+			(xy 121.92 123.19) (xy 121.92 135.89)
 		)
 		(stroke
@@
 		(pts
 			(xy 176.53 92.71) (xy 176.53 104.14)
-		)
-		(stroke
-			(width 0)
-			(type default)
-		)
-	)
-	(wire
-		(pts
-			(xy 121.92 110.49) (xy 121.92 111.76)
 		)
 		(stroke
@@
 	)
 	(symbol
-		(lib_id "Sensor_Optical:BP103")
-		(at 124.46 116.84 180)
-		(unit 1)
-		(exclude_from_sim no)
-		(in_bom yes)
-		(on_board yes)
-		(dnp no)
-		(fields_autoplaced yes)
-		(property "Reference" "Q1"
-			(at 119.38 116.3192 0)
-			(effects
-				(font
-					(size 1.27 1.27)
-				)
-				(justify left)
-			)
-		)
-		(property "Value" "BP103"
-			(at 119.38 118.8592 0)
-			(effects
-				(font
-					(size 1.27 1.27)
-				)
-				(justify left)
-			)
-		)
-		(property "Footprint" "Package_TO_SOT_THT:TO-18-3_Lens"
-			(at 119.253 113.284 0)
-			(effects
-				(font
-					(size 1.27 1.27)
-				)
-				(justify left)
-				(hide yes)
-			)
-		)
-		(property "Datasheet" "http://www.osram-os.com/Graphics/XPic3/00101777_0.pdf/BP"
-			(at 124.46 116.84 0)
-			(effects
-				(font
-					(size 1.27 1.27)
-				)
-				(hide yes)
-			)
-		)
-		(property "Description" "NPN Phototransistor"
-			(at 124.46 116.84 0)
-			(effects
-				(font
-					(size 1.27 1.27)
-				)
-				(hide yes)
-			)
-		)
-		(pin "1"
-		)
-		(pin "2"
-		)
-		(pin "3"
-		)
-		(instances
-			(project ""
-				(path "/063249a1-dd82-4aba-aeae-aae1f466d57b"
-					(reference "Q1")
-					(unit 1)
-				)
-			)
-		)
-	)
-	(symbol
 		(lib_id "Simulation_SPICE:NPN")
 		(at 152.4 110.49 0)
@@
 	(symbol
 		(lib_id "Device:R_Photo")
-		(at 121.92 107.95 0)
+		(at 121.92 106.68 0)
 		(unit 1)
 		(exclude_from_sim no)
@@
 		(fields_autoplaced yes)
 		(property "Reference" "R3"
-			(at 124.46 106.6799 0)
+			(at 124.46 105.4099 0)
 			(effects
 				(font
@@
 		)
 		(property "Value" "R_Photo"
-			(at 124.46 109.2199 0)
+			(at 124.46 107.9499 0)
 			(effects
 				(font
@@
 		)
 		(property "Footprint" "OptoDevice:R_LDR_5.1x4.3mm_P3.4mm_Vertical"
-			(at 123.19 114.3 90)
+			(at 123.19 113.03 90)
 			(effects
 				(font
@@
 		)
 		(property "Datasheet" "~"
-			(at 121.92 109.22 0)
+			(at 121.92 107.95 0)
 			(effects
 				(font
@@
 		)
 		(property "Description" "Photoresistor"
-			(at 121.92 107.95 0)
+			(at 121.92 106.68 0)
 			(effects
 				(font
@@
 					(unit 1)
 				)
+			)
+		)
+	)
+	(symbol
+		(lib_id "Sensor_Optical:BP103")
+		(at 124.46 118.11 180)
+		(unit 1)
+		(exclude_from_sim no)
+		(in_bom yes)
+		(on_board yes)
+		(dnp no)
+		(fields_autoplaced yes)
+		(property "Reference" "Q4"
+			(at 119.38 117.5892 0)
+			(effects
+				(font
+					(size 1.27 1.27)
+				)
+				(justify left)
+			)
+		)
+		(property "Value" "BP103"
+			(at 119.38 120.1292 0)
+			(effects
+				(font
+					(size 1.27 1.27)
+				)
+				(justify left)
+			)
+		)
+		(property "Footprint" "Package_TO_SOT_THT:TO-18-3_Lens"
+			(at 119.253 114.554 0)
+			(effects
+				(font
+					(size 1.27 1.27)
+				)
+				(justify left)
+				(hide yes)
+			)
+		)
+		(property "Datasheet" "http://www.osram-os.com/Graphics/XPic3/00101777_0.pdf/BP"
+			(at 124.46 118.11 0)
+			(effects
+				(font
+					(size 1.27 1.27)
+				)
+				(hide yes)
+			)
+		)
+		(property "Description" "NPN Phototransistor"
+			(at 124.46 118.11 0)
+			(effects
+				(font
+					(size 1.27 1.27)
+				)
+				(hide yes)
+			)
+		)
+		(pin "1"
+		)
+		(pin "2"
+		)
+		(pin "3"
+		)
+		(instances
+			(project "nano"
+				(path "/063249a1-dd82-4aba-aeae-aae1f466d57b"
+					(reference "Q4")
+					(unit 1)
+				)
